Commit message: renamed pkg

File: DRIMS_dice_demo/xacro/Extra/dice.urdf (robot description, URDF)
Before this commit: robot dice, 1 links, 0 joints
Links:
- link dice: geometry collision mesh filename=package://DRIMS_dice_demo/meshes/Dice/Die-OBJ.obj scale=0.03 0.03 0.03; visual mesh filename=package://DRIMS_dice_demo/meshes/Dice/Die-OBJ.obj scale=0.03 0.03 0.03

File: DRIMS_dice_demo/xacro/Extra/table.xacro (robot description, xacro)
@@ -25,5 +25,5 @@
                 <origin rpy="0 0 0" xyz="0 0 0.6"/>
                 <geometry>
-                    <mesh filename="package://irim_ss_pkg/meshes/Extra/table.obj" scale="1.5 1 0.05"/>
+                    <mesh filename="package://DRIMS_dice_demo/meshes/Extra/table.obj" scale="1.5 1 0.05"/>
                 </geometry>
                 <!-- <material name="Gazebo/Yellow"/> -->
@@ -32,5 +32,5 @@
                 <origin rpy="0 0 0" xyz="0 0 0.6"/>
                 <geometry>
-                    <mesh filename="package://irim_ss_pkg/meshes/Extra/table.obj" scale="1.5 1 0.05"/>
+                    <mesh filename="package://DRIMS_dice_demo/meshes/Extra/table.obj" scale="1.5 1 0.05"/>
                 </geometry>
                 <!-- <material name="Gazebo/Yellow"/> -->
@@ -45,5 +45,5 @@
                 <origin rpy="0 0 0" xyz="-0.65 -0.4 0.29"/>
                 <geometry>
-                    <mesh filename="package://irim_ss_pkg/meshes/Extra/table.obj" scale="0.1 0.1 0.58"/>
+                    <mesh filename="package://DRIMS_dice_demo/meshes/Extra/table.obj" scale="0.1 0.1 0.58"/>
                 </geometry>
                 <!-- <material name="white">
@@ -54,5 +54,5 @@
                 <origin rpy="0 0 0" xyz="-0.65 0.4 0.29"/>
                 <geometry>
-                    <mesh filename="package://irim_ss_pkg/meshes/Extra/table.obj" scale="0.1 0.1 0.58"/>
+                    <mesh filename="package://DRIMS_dice_demo/meshes/Extra/table.obj" scale="0.1 0.1 0.58"/>
                 </geometry>
                 <!-- <material name="white">
@@ -63,5 +63,5 @@
                 <origin rpy="0 0 0" xyz="0.65 -0.4 0.29"/>
                 <geometry>
-                    <mesh filename="package://irim_ss_pkg/meshes/Extra/table.obj" scale="0.1 0.1 0.58"/>
+                    <mesh filename="package://DRIMS_dice_demo/meshes/Extra/table.obj" scale="0.1 0.1 0.58"/>
                 </geometry>
                 <!-- <material name="white">
@@ -72,5 +72,5 @@
                 <origin rpy="0 0 0" xyz="0.65 0.4 0.29"/>
                 <geometry>
-                    <mesh filename="package://irim_ss_pkg/meshes/Extra/table.obj" scale="0.1 0.1 0.58"/>
+                    <mesh filename="package://DRIMS_dice_demo/meshes/Extra/table.obj" scale="0.1 0.1 0.58"/>
                 </geometry>
             </visual>

File: DRIMS_dice_demo/xacro/irim_yumi.urdf.xacro (robot description, xacro)
@@ -12,29 +12,29 @@
     <!-- Robot -->
     <!-- Import Rviz colors -->
-    <xacro:include filename="$(find robots_description)/Util/materials.xacro" />
+    <xacro:include filename="$(find omnicore_description)/Util/materials.xacro" />
     <!-- Import utilities -->
-    <xacro:include filename="$(find robots_description)/Util/utilities.xacro" />
+    <xacro:include filename="$(find omnicore_description)/Util/utilities.xacro" />
     <!-- Import the table -->
-    <xacro:include filename="$(find irim_ss_pkg)/xacro/Extra/table.xacro" />
+    <xacro:include filename="$(find DRIMS_dice_demo)/xacro/Extra/table.xacro" />
     <xacro:table parent="world" >
         <origin xyz="0 0 0" rpy="0 0 0" />
     </xacro:table>
     <!-- Import the table -->
-    <xacro:include filename="$(find irim_ss_pkg)/xacro/Extra/camera_stand.xacro" />
+    <xacro:include filename="$(find DRIMS_dice_demo)/xacro/Extra/camera_stand.xacro" />
     <xacro:camera_stand parent="base_link_table" >
         <origin xyz="0.0 0.4 0.65" rpy="0 0 0" />
     </xacro:camera_stand>
     <!-- Import the surface -->
-    <xacro:include filename="$(find irim_ss_pkg)/xacro/Extra/surface.xacro" />
+    <xacro:include filename="$(find DRIMS_dice_demo)/xacro/Extra/surface.xacro" />
     <xacro:surface parent="single_yumi_base_link" >
         <origin xyz="-0.03 0.33 0.08" rpy="0 0 0" />
     </xacro:surface>
     <!--Import the single yumi macro -->
-    <xacro:include filename="$(find robots_description)/xacro/YumiSingleArm/single_yumi.xacro" />
+    <xacro:include filename="$(find omnicore_description)/xacro/YumiSingleArm/single_yumi.xacro" />
     <xacro:single_yumi parent="base_link_table" hardware_interface="${hardware_interface}">
         <origin xyz="-0.3 0 0.6" rpy="0 0 -1.57" />
     </xacro:single_yumi>
     <!--Import the yumi servo gripper macro -->
-    <xacro:include filename="$(find robots_description)/Grippers/YumiServoGripper/yumi_servo_gripper.xacro" />
+    <xacro:include filename="$(find omnicore_description)/Grippers/YumiServoGripper/yumi_servo_gripper.xacro" />
     <!-- Gripper -->
     <xacro:yumi_servo_gripper name="gripper" parent="link_7" hardware_interface="${gripper_interface}" fake_execution="'true'">
