Commit message: marco : fixed naming convention

File: drims_dice_demo/xacro/Extra/dice.urdf (robot description, URDF)
Before this commit: robot dice, 1 links, 0 joints
Links:
- link dice: geometry collision mesh filename=package://drims_dice_demo/meshes/Dice/Die-OBJ.obj scale=0.03 0.03 0.03; visual mesh filename=package://drims_dice_demo/meshes/Dice/Die-OBJ.obj scale=0.03 0.03 0.03

File: drims_dice_demo/xacro/Extra/table.xacro (robot description, xacro)
@@ -25,5 +25,5 @@
                 <origin rpy="0 0 0" xyz="0 0 0.6"/>
                 <geometry>
-                    <mesh filename="package://DRIMS_dice_demo/meshes/Extra/table.obj" scale="1.5 1 0.05"/>
+                    <mesh filename="package://drims_dice_demo/meshes/Extra/table.obj" scale="1.5 1 0.05"/>
                 </geometry>
                 <!-- <material name="Gazebo/Yellow"/> -->
@@ -32,5 +32,5 @@
                 <origin rpy="0 0 0" xyz="0 0 0.6"/>
                 <geometry>
-                    <mesh filename="package://DRIMS_dice_demo/meshes/Extra/table.obj" scale="1.5 1 0.05"/>
+                    <mesh filename="package://drims_dice_demo/meshes/Extra/table.obj" scale="1.5 1 0.05"/>
                 </geometry>
                 <!-- <material name="Gazebo/Yellow"/> -->
@@ -45,5 +45,5 @@
                 <origin rpy="0 0 0" xyz="-0.65 -0.4 0.29"/>
                 <geometry>
-                    <mesh filename="package://DRIMS_dice_demo/meshes/Extra/table.obj" scale="0.1 0.1 0.58"/>
+                    <mesh filename="package://drims_dice_demo/meshes/Extra/table.obj" scale="0.1 0.1 0.58"/>
                 </geometry>
                 <!-- <material name="white">
@@ -54,5 +54,5 @@
                 <origin rpy="0 0 0" xyz="-0.65 0.4 0.29"/>
                 <geometry>
-                    <mesh filename="package://DRIMS_dice_demo/meshes/Extra/table.obj" scale="0.1 0.1 0.58"/>
+                    <mesh filename="package://drims_dice_demo/meshes/Extra/table.obj" scale="0.1 0.1 0.58"/>
                 </geometry>
                 <!-- <material name="white">
@@ -63,5 +63,5 @@
                 <origin rpy="0 0 0" xyz="0.65 -0.4 0.29"/>
                 <geometry>
-                    <mesh filename="package://DRIMS_dice_demo/meshes/Extra/table.obj" scale="0.1 0.1 0.58"/>
+                    <mesh filename="package://drims_dice_demo/meshes/Extra/table.obj" scale="0.1 0.1 0.58"/>
                 </geometry>
                 <!-- <material name="white">
@@ -72,5 +72,5 @@
                 <origin rpy="0 0 0" xyz="0.65 0.4 0.29"/>
                 <geometry>
-                    <mesh filename="package://DRIMS_dice_demo/meshes/Extra/table.obj" scale="0.1 0.1 0.58"/>
+                    <mesh filename="package://drims_dice_demo/meshes/Extra/table.obj" scale="0.1 0.1 0.58"/>
                 </geometry>
             </visual>

File: drims_dice_demo/xacro/irim_yumi.urdf.xacro (robot description, xacro)
@@ -16,15 +16,15 @@
     <xacro:include filename="$(find omnicore_description)/Util/utilities.xacro" />
     <!-- Import the table -->
-    <xacro:include filename="$(find DRIMS_dice_demo)/xacro/Extra/table.xacro" />
+    <xacro:include filename="$(find drims_dice_demo)/xacro/Extra/table.xacro" />
     <xacro:table parent="world" >
         <origin xyz="0 0 0" rpy="0 0 0" />
     </xacro:table>
     <!-- Import the table -->
-    <xacro:include filename="$(find DRIMS_dice_demo)/xacro/Extra/camera_stand.xacro" />
+    <xacro:include filename="$(find drims_dice_demo)/xacro/Extra/camera_stand.xacro" />
     <xacro:camera_stand parent="base_link_table" >
         <origin xyz="0.0 0.4 0.65" rpy="0 0 0" />
     </xacro:camera_stand>
     <!-- Import the surface -->
-    <xacro:include filename="$(find DRIMS_dice_demo)/xacro/Extra/surface.xacro" />
+    <xacro:include filename="$(find drims_dice_demo)/xacro/Extra/surface.xacro" />
     <xacro:surface parent="single_yumi_base_link" >
         <origin xyz="-0.03 0.33 0.08" rpy="0 0 0" />
