Commit message: Added choice for GoFa and YuMi single arm robot.

File: drims_dice_demo/xacro/Extra/camera_stand.xacro (robot description, xacro)
@@ -58,5 +58,5 @@
                     <box size="0.01 0.01 0.01"/>
                 </geometry>
-                <material name="red"/>
+                <material name="Red"/>
             </visual>
             <inertial>

Commit message: Modified simulated and real enviroment with camera stand and surface for Gofa arm.

File: drims_dice_demo/xacro/Extra/camera_stand.xacro (robot description, xacro)
@@ -3,5 +3,5 @@
     <xacro:macro name="camera_stand" params="parent *origin">
         <xacro:property name="base_height" value="0.88" />
-        <xacro:property name="holder_length" value="0.3" />
+        <xacro:property name="holder_length" value="0.55" />
         <joint name="joint_camera_stand_robot" type="fixed">
             <xacro:insert_block name="origin"/>
@@ -24,5 +24,5 @@
                 <origin xyz="0 0 ${base_height/2}" rpy="0 0 0"/>
                 <geometry>
-                    <box size="0.04 0.04 ${base_height}" />
+                    <box size="0.1 0.1 ${base_height}" />
                 </geometry>
             </collision>
@@ -43,5 +43,5 @@
                 <origin xyz="0 0 ${holder_length/2}" rpy="0 0 0"/>
                 <geometry>
-                    <box size="0.1 0.1 ${holder_length}" />
+                    <box size="0.15 0.15 ${holder_length}" />
                 </geometry>
             </collision>
@@ -67,5 +67,5 @@
         </link>
         <joint name="joint_camera_link" type="fixed">
-            <origin xyz="0.0 0.0 ${holder_length + 0.1}" rpy="-${pi/2} 0 -3.14 " />
+            <origin xyz="0.0 0.0 ${holder_length - 0.12}" rpy="-${pi/2} 0 -3.14 " />
             <parent link="camera_holder" />
             <child link="ext_camera_link" />

File: drims_dice_demo/xacro/Extra/surface.xacro (robot description, xacro)
@@ -3,6 +3,6 @@
     <!-- 72 52 2 -->
     <xacro:macro name="surface" params="parent *origin">
-        <xacro:property name="base_height" value="0.6" />
-        <xacro:property name="base_width" value="0.4" />
+        <xacro:property name="base_height" value="0.75" />
+        <xacro:property name="base_width" value="0.52" />
         <joint name="joint_surface_robot" type="fixed">
             <xacro:insert_block name="origin"/>
@@ -22,5 +22,5 @@
                 <origin xyz="0 0 0" rpy="0 0 0"/>
                 <geometry>
-                    <box size="${base_height} ${base_width} 0.1" />
+                    <box size="${base_height} ${base_width} 0.005" />
                 </geometry>
             </visual>
@@ -28,5 +28,5 @@
                 <origin xyz="0 0 0" rpy="0 0 0"/>
                 <geometry>
-                    <box size="${base_height} ${base_width} 0.1" />
+                    <box size="${base_height} ${base_width} 0.005" />
                 </geometry>
             </collision>

File: drims_dice_demo/xacro/Extra/table.xacro (robot description, xacro)
@@ -25,5 +25,5 @@
                 <origin rpy="0 0 0" xyz="0 0 0.6"/>
                 <geometry>
-                    <mesh filename="package://drims_dice_demo/meshes/Extra/table.obj" scale="1.5 1 0.05"/>
+                    <mesh filename="package://drims_dice_demo/meshes/Extra/table.obj" scale="1.9 1.3 0.05"/>
                 </geometry>
                 <!-- <material name="Gazebo/Yellow"/> -->

File: drims_dice_demo/xacro/robot_arm.urdf.xacro (robot description, xacro)
@@ -81,9 +81,9 @@
         <!-- Include surface -->
         <xacro:surface parent="${robot}_base_link">
-            <origin xyz="-0.03 -0.50 0.1" rpy="0 0 0" />
+            <origin xyz="0.145 -0.77 0.0" rpy="0 0 0" />
         </xacro:surface>
         <!-- Include camera stand -->
         <xacro:camera_stand parent="base_link_surface">
-            <origin xyz="0.325 0.0 0.0" rpy="0 0 ${-PI / 2.0}" />
+            <origin xyz="0.355 0.0 0.0" rpy="0 0 ${-PI / 2.0}" />
         </xacro:camera_stand>
         <xacro:gofa parent="base_link_table" child="${robot}_base_link"
