Commit message: Modified scene in simulation

File: drims_dice_demo/xacro/robot_arm.urdf.xacro (robot description, xacro)
@@ -37,14 +37,14 @@
         <origin xyz="0 0 0" rpy="0 0 0" />
     </xacro:table>
-    <!-- Include camera stand -->
-    <xacro:camera_stand parent="base_link_table">
-        <origin xyz="0.0 0.4 0.65" rpy="0 0 0" />
-    </xacro:camera_stand>
-    <!-- Include surface -->
-    <xacro:surface parent="${robot}_base_link">
-        <origin xyz="-0.03 0.33 0.08" rpy="0 0 0" />
-    </xacro:surface>
     <!-- Choose between gofa and yumi_single_arm -->
     <xacro:if value="${robot == 'yumi'}">
+        <!-- Include camera stand -->
+        <xacro:camera_stand parent="base_link_table">
+            <origin xyz="0.0 0.4 0.65" rpy="0 0 0" />
+        </xacro:camera_stand>
+        <!-- Include surface -->
+        <xacro:surface parent="${robot}_base_link">
+            <origin xyz="-0.03 -0.33 0.08" rpy="0 0 0" />
+        </xacro:surface>
         <xacro:single_yumi parent="base_link_table" child="${robot}_base_link"
             hardware_interface="${hardware_interface}">
@@ -58,7 +58,15 @@
     </xacro:if>
     <xacro:if value="${robot == 'gofa'}">
+        <!-- Include surface -->
+        <xacro:surface parent="${robot}_base_link">
+            <origin xyz="-0.03 -0.50 0.1" rpy="0 0 0" />
+        </xacro:surface>
+        <!-- Include camera stand -->
+        <xacro:camera_stand parent="base_link_surface">
+            <origin xyz="0.325 0.0 0.0" rpy="0 0 ${-PI / 2.0}" />
+        </xacro:camera_stand>
         <xacro:gofa parent="base_link_table" child="${robot}_base_link"
             hardware_interface="${hardware_interface}">
-            <origin xyz="-0.3 0 0.627" rpy="0 0 -1.57" />
+            <origin xyz="-0.6 0 0.627" rpy="0 0 1.57" />
         </xacro:gofa>
         <xacro:egk_40_gazebo
@@ -66,5 +74,5 @@
             parent="flange"
             px="0.0" py="0.0" pz="0.011"
-            rx="${pi / 2.0}" ry="0.0" rz="0.0"
+            rx="${pi / 2.0}" ry="0.0" rz="${pi / 6.0}"
             hardware_interface="$(arg gripper_interface)" />
     </xacro:if>

Commit message: Modified scene in simulation.

File: drims_dice_demo/xacro/robot_arm.urdf.xacro (robot description, xacro)
@@ -39,15 +39,15 @@
     <!-- Choose between gofa and yumi_single_arm -->
     <xacro:if value="${robot == 'yumi'}">
-        <!-- Include camera stand -->
-        <xacro:camera_stand parent="base_link_table">
-            <origin xyz="0.0 0.4 0.65" rpy="0 0 0" />
-        </xacro:camera_stand>
         <!-- Include surface -->
         <xacro:surface parent="${robot}_base_link">
-            <origin xyz="-0.03 -0.33 0.08" rpy="0 0 0" />
+            <origin xyz="-0.03 -0.40 0.1" rpy="0 0 0" />
         </xacro:surface>
+        <!-- Include camera stand -->
+        <xacro:camera_stand parent="base_link_surface">
+            <origin xyz="0.325 0.0 0.0" rpy="0 0 ${-PI / 2.0}" />
+        </xacro:camera_stand>
         <xacro:single_yumi parent="base_link_table" child="${robot}_base_link"
             hardware_interface="${hardware_interface}">
-            <origin xyz="-0.3 0 0.6" rpy="0 0 -1.57" />
+            <origin xyz="-0.6 0 0.6" rpy="0 0 1.57" />
         </xacro:single_yumi>
         <!-- Smart Gripper -->

Commit message: Fixes YUMI

File: drims_dice_demo/xacro/robot_arm.urdf.xacro (robot description, xacro)
@@ -38,4 +38,5 @@
     </xacro:table>
     <!-- Choose between gofa and yumi_single_arm -->
+    <!-- For real yumi -->
     <xacro:if value="${robot == 'yumi_single_arm'}">
         <!-- Include surface -->
@@ -48,4 +49,24 @@
         </xacro:camera_stand>
         <xacro:single_yumi parent="base_link_table" child="yumi_base_link"
+            hardware_interface="${hardware_interface}">
+            <origin xyz="-0.6 0 0.6" rpy="0 0 1.57" />
+        </xacro:single_yumi>
+        <!-- Smart Gripper -->
+        <xacro:yumi_servo_gripper name="gripper" parent="link_7"
+            hardware_interface="${gripper_interface}">
+            <origin xyz="0 0 0.007" rpy="0 0 ${PI}" />
+        </xacro:yumi_servo_gripper>
+    </xacro:if>
+    <!-- For fake yumi -->
+    <xacro:if value="${robot == 'yumi'}">
+        <!-- Include surface -->
+        <xacro:surface parent="{robot}_base_link">
+            <origin xyz="-0.03 -0.40 0.1" rpy="0 0 0" />
+        </xacro:surface>
+        <!-- Include camera stand -->
+        <xacro:camera_stand parent="base_link_surface">
+            <origin xyz="0.325 0.0 0.0" rpy="0 0 ${-PI / 2.0}" />
+        </xacro:camera_stand>
+        <xacro:single_yumi parent="base_link_table" child="{robot}_base_link"
             hardware_interface="${hardware_interface}">
             <origin xyz="-0.6 0 0.6" rpy="0 0 1.57" />

Commit message: minor changes

File: drims_dice_demo/xacro/robot_arm.urdf.xacro (robot description, xacro)
@@ -66,5 +66,5 @@
         <!-- Include camera stand -->
         <xacro:camera_stand parent="base_link_surface">
-            <origin xyz="0.325 0.0 0.0" rpy="0 0 ${-PI / 2.0}" />
+            <origin xyz="0.425 0.0 0.0" rpy="0 0 ${-PI / 2.0}" />
         </xacro:camera_stand>
         <xacro:single_yumi parent="base_link_table" child="{robot}_base_link"
